Commit message: Update robot.urdf

File: catkin_ws/src/lab2/urdf/robot.urdf (robot description, URDF)
Before this commit: robot roBOT, 6 links, 5 joints
Links:
- added link join3; visual cylinder length=0.6 radius=0.2
Joints:
- added joint link3_join3: type fixed, parent link3, child join3, origin xyz=0 ${params['thirdRow']['len']} 0 rpy=0 0 0, axis 0 0 1, limit lower=-3.14  upper=3.14 effort=1000.0 velocity=0.5
- joint join2_link3: origin xyz=0 ${params['secondRow']['len']} 0  rpy=0 0 0 -> xyz=0 0 0  rpy=0 0 0
- joint link2_join2: origin xyz=0 0 0 rpy=0 0 0 -> xyz=0 ${params['secondRow']['len']} 0 rpy=0 0 0

Commit message: Wersja Rafał po majówce urdf

File: catkin_ws/src/lab2/urdf/robot.urdf (robot description, URDF)
Before this commit: robot roBOT, 7 links, 6 joints
Joints:
- joint base_link1: origin xyz=0 0 0 rpy=0 0 0 -> xyz=0 0 0 rpy=${params['firstRow']['rpy']}
- joint join1_link2: origin xyz=0 0 0 rpy=0 0 0 -> xyz=0 0 0 rpy=${params['secondRow']['rpy']}
- joint join2_link3: origin xyz=0 0 0  rpy=0 0 0 -> xyz=0 0 0  rpy=${params['thirdRow']['rpy']}
- joint link2_join2: origin xyz=0 ${params['secondRow']['len']} 0 rpy=0 0 0 -> xyz=${params['secondRow']['len']} 0 0 rpy=0 0 0
- joint link3_join3: origin xyz=0 ${params['thirdRow']['len']} 0 rpy=0 0 0 -> xyz=${params['thirdRow']['len']} 0 0 rpy=0 0 0

Commit message: add 3rd project

File: catkin_ws/src/lab2/urdf/robot.urdf (robot description, URDF)
Before this commit: robot roBOT, 7 links, 6 joints
Links:
- removed link join3
Joints:
- removed joint link3_join3
- joint base_link1: origin xyz=0 0 0 rpy=${params['firstRow']['rpy']} -> xyz=0 0 0 rpy=0 0 0
- joint join1_link2: origin xyz=0 0 0 rpy=${params['secondRow']['rpy']} -> xyz=0 0 0 rpy=0 0 0
- joint join2_link3: origin xyz=0 0 0  rpy=${params['thirdRow']['rpy']} -> xyz=0 ${params['secondRow']['len']} 0  rpy=0 0 0
- joint link2_join2: origin xyz=${params['secondRow']['len']} 0 0 rpy=0 0 0 -> xyz=0 0 0 rpy=0 0 0
